File: μTeslaCoil.kicad_sch (KiCad schematic)
At the start: 64 parts, among them J10 T2, J12 12V, J2 PRI, J3 FB, J4 SW, J6 SW, J7 T4, J8 T3, J9 T1, Q1 NCE0224K, Q2 NCE0224K, Q3 NCE0224K, U1 XL6009, U2 NE555D

Commit message: rev 1.3
Parts:
- removed C11, C12: 1u 100V, Capacitor_SMD:C_1206_3216Metric, symbol Device:C
- removed D2: 12V, Diode_SMD:D_SOD-123, symbol Device:D_Zener
- removed D5, D6: 1N4148, Diode_SMD:D_SOD-123, symbol Device:D
- removed J12: 12V, TestPoint:TestPoint_Pad_1.0x1.0mm, symbol Connector_Generic:Conn_01x01
- removed R10: 47k, Resistor_SMD:R_0805_2012Metric, symbol Device:R
- removed R6: 4.7k, Resistor_SMD:R_0805_2012Metric, symbol Device:R
- removed R9: 470, Resistor_SMD:R_0805_2012Metric, symbol Device:R
- added C15: 1u 100V, Capacitor_SMD:C_1206_3216Metric, symbol Device:C
- added D10, D2, D3: 180V, Diode_SMD:D_SMB, symbol Device:D_TVS
- added D6, D7: 1N5819, Diode_SMD:D_SOD-123, symbol Device:D_Schottky
- added D8, D9: 1N4148, Diode_SMD:D_SOD-123, symbol Device:D
- added RV3: 10k, Potentiometer_THT:Potentiometer_ACP_CA9-H2,5_Horizontal, symbol Device:R_Potentiometer
- H7: renamed from H4; value GND -> 12V
- R4: value 15k -> 47k
- R5: value 6.8k -> 470
- RV1: footprint Potentiometer_THT:Potentiometer_ACP_CA9-H2,5_Horizontal -> Potentiometer_THT:Potentiometer_Bourns_3296W_Vertical
- renumbered C2 to C1, C9 to C10, C10 to C11, C17 to C12, C14 to C13, C15 to C14, C3 to C2, C6 to C3, C1 to C4, C7 to C5, C4 to C6, C5 to C7, C18 to C8, C8 to C9, D3 to D4, D4 to D5, H11 to H1, H7 to H10, H8 to H11, H9 to H2, H10 to H3, H1 to H4, H2 to H5, H3 to H6, H5 to H8, H6 to H9, J2 to J1, J3 to J2, J7 to J3, J8 to J4, J9 to J5, J10 to J6, J4 to J7, J6 to J8, L2 to L1, L3 to L2, L1 to L3, R11 to R6
Connections:
- net +12V: now also H7.1, R4.2, RV1.3
- net GND: now also C10.2, C11.2, C9.2, D4.1 (A1), D5.1 (A1), Q1.3 (S), Q2.3 (S), RV1.1, C15.2, D10.2 (A2), D2.1 (A1), D3.2 (A2); no longer H7.1
- net VDD: no longer R4.1
- net at D5.2 (A2), J6.1 (Pin_1), Q2.1 (G): now also RV1.2, D7.2 (A); no longer R5.2
- net at C16.1, U2.2 (TR), U2.6 (THR): now also D8.1 (K), D9.2 (A)
- net at C11.1, J1.1 (Pin_1), L2.2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: now also D3.1 (A1)
- net at R5.1: now also RV3.2, RV3.3; no longer R4.2
- net at RV2.1, U2.7 (DIS): now also D8.2 (A), RV3.1; no longer RV1.2, RV1.3
- net at RV2.2, RV2.3: now also R4.1
- net at C10.1, C3.1, C5.1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: now also D2.2 (A2)
- net interrupter: now reaches R7.2, U2.3 (Q)
- net at D4.2 (A2), J5.1 (Pin_1), Q1.1 (G): now also D6.2 (A)
- new net: D9.1 (K), R5.2
- new net: C15.1, D10.1 (A1), D6.1 (K), D7.1 (K), Q3.2 (D)
Other:
- title: Mini Tesla -> μTeslaCoil
- moved on the sheet: C1, C10, C11, C12, C13, C14, C16, C2, C3, C5, C9, D4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
