File: μTeslaCoil.kicad_pcb (KiCad board)
At the start: 2 copper layers, 203.6 x 138.7 mm, 366 parts, among them J10 T2, J12 12V, J2 PRI, J4 SW, J6 SW, J8 T3, J9 T1, Q1 NCE0224K, Q2 NCE0224K, Q3 NCE0224K, U1 XL6009, U2 NE555D

Commit message: small clean-up
Parts:
- removed the G*** at (116.3, 18.5)
- removed the G*** at (79.4, 19.3)

Commit message: rev 1.3
Parts:
- removed the C1 at (86.3, 115.7)
- removed the C1 at (86.3, 80.2)
- removed the C1 at (44.0, 115.7)
- removed the C1 at (44.0, 80.2)
- removed the C10 at (171.9, 73.7)
- removed the C10 at (171.9, 101.1)
- removed the C10 at (171.9, 128.5)
- removed the C11 at (165.9, 87.7)
- removed the C11 at (165.9, 115.1)
- removed the C11 at (165.9, 142.5)
- removed the C11 at (94.0, 42.9)
- removed the C12 at (190.1, 142.5)
- removed the C12 at (190.1, 87.7)
- removed the C12 at (190.1, 115.1)
- removed the C12 at (118.1, 42.9)
- removed the C14 at (208.1, 119.9)
- removed the C14 at (208.1, 147.3)
- removed the C14 at (208.1, 92.5)
- removed the C15 at (201.5, 145.5)
- removed the C15 at (201.5, 90.7)
- removed the C15 at (201.5, 118.1)
- removed the C16 at (214.5, 87.9)
- removed the C16 at (214.5, 142.7)
- removed the C16 at (214.5, 115.3)
- removed C17 (x3): 100n, Capacitor_SMD:C_0805_2012Metric
- removed C18 (x5): 1000u, Capacitor_THT:CP_Radial_D16.0mm_P7.50mm
- removed the C2 at (159.3, 135.6)
- removed the C2 at (159.3, 108.2)
- removed the C2 at (159.3, 80.8)
- removed the C3 at (159.3, 118.4)
- removed the C3 at (159.3, 91.0)
- removed the C3 at (159.3, 145.8)
- removed the C4 at (43.2, 83.8)
- removed the C4 at (43.2, 119.3)
- removed the C4 at (85.6, 83.8)
- removed the C4 at (85.6, 119.3)
- removed the C5 at (97.6, 139.2)
- removed the C5 at (97.6, 103.7)
- removed the C5 at (55.2, 139.2)
- removed the C5 at (55.2, 103.7)
- removed the C6 at (150.2, 92.5)
- removed the C6 at (150.2, 147.3)
- removed the C6 at (150.2, 119.9)
- removed the C7 at (150.2, 122.6)
- removed the C7 at (150.2, 150.0)
- removed the C7 at (150.2, 95.2)
- removed the C8 at (180.6, 128.5)
- removed the C8 at (180.6, 73.7)
- removed the C8 at (180.6, 101.1)
- removed the C9 at (171.8, 142.5)
- removed the C9 at (171.8, 87.7)
- removed the C9 at (171.8, 115.1)
- removed the D1 at (64.8, 102.0)
- removed the D1 at (107.2, 102.0)
- removed the D1 at (64.8, 137.5)
- removed the D1 at (107.2, 137.5)
- removed the D2 at (169.8, 140.8)
- removed the D2 at (169.8, 86.0)
- removed the D2 at (97.8, 41.2)
- removed the D2 at (169.8, 113.4)
- removed the D3 at (178.3, 120.2)
- removed the D3 at (178.3, 147.6)
- removed the D3 at (178.3, 92.8)
- removed the D4 at (178.3, 78.8)
- removed the D4 at (178.3, 106.2)
- removed the D4 at (178.3, 133.6)
- removed the D5 at (207.5, 116.1)
- removed the D5 at (207.5, 143.5)
- removed the D5 at (135.5, 43.9)
- removed the D5 at (207.5, 88.7)
- removed the D6 at (209.9, 88.7)
- removed the D6 at (137.9, 43.9)
- removed the D6 at (209.9, 116.1)
- removed the D6 at (209.9, 143.5)
- removed the G*** at (150.3, 103.4)
- removed the G*** at (184.2, 113.4)
- removed the G*** at (103.4, 109.4) (x2)
- removed the G*** at (186.7, 79.2)
- removed the G*** at (186.7, 106.6)
- removed the G*** at (186.7, 134.0)
- removed the G*** at (150.3, 130.8)
- removed the G*** at (61.0, 109.4) (x2)
- removed the G*** at (204.7, 121.9)
- removed the G*** at (103.4, 144.9) (x2)
- removed the G*** at (103.4, 136.5)
- removed the G*** at (61.0, 144.9) (x2)
- removed the G*** at (183.0, 139.6)
- removed the G*** at (111.0, 40.0)
- removed the G*** at (183.0, 112.2)
- removed the G*** at (183.0, 84.8)
- removed the G*** at (150.3, 76.0)
- removed the G*** at (52.3, 55.5)
- removed the G*** at (204.7, 149.3)
- removed the G*** at (103.4, 101.0)
- removed the G*** at (61.0, 101.0)
- removed the G*** at (61.0, 136.5)
- removed the G*** at (204.7, 94.5)
- removed the G*** at (184.2, 140.8)
- removed the G*** at (184.2, 86.0)
- removed the H1 at (143.1, 102.4)
- removed the H1 at (143.1, 129.8)
- removed the H1 at (143.1, 75.0)
- removed the H10 at (79.0, 143.1)
- removed the H10 at (36.6, 143.1)
- removed the H10 at (36.6, 107.6)
- removed the H10 at (79.0, 107.6)
- removed the H11 at (36.6, 115.7)
- removed the H11 at (79.0, 80.2)
- removed the H11 at (36.6, 80.2)
- removed the H11 at (79.0, 115.7)
- removed the H2 at (143.1, 149.1)
- removed the H2 at (143.1, 121.7)
- removed the H2 at (143.1, 94.3)
- removed the H3 at (213.2, 149.1)
- removed the H3 at (213.2, 121.7)
- removed the H3 at (213.2, 94.3)
- removed the H4 at (213.2, 129.8)
- removed the H4 at (213.2, 102.4)
- removed the H4 at (213.2, 75.0)
- removed the H5 at (152.1, 140.6)
- removed the H5 at (152.1, 113.2)
- removed the H5 at (152.1, 85.8)
- removed the H6 at (159.7, 85.8)
- removed the H6 at (159.7, 113.2)
- removed the H6 at (159.7, 140.6)
- removed the H7 at (70.9, 143.1)
- removed the H7 at (113.3, 143.1)
- removed the H7 at (70.9, 107.6)
- removed the H7 at (113.3, 107.6)
- removed the H8 at (113.3, 80.2)
- removed the H8 at (113.3, 115.7)
- removed the H8 at (70.9, 80.2)
- removed the H8 at (70.9, 115.7)
- removed the H9 at (92.2, 80.2)
- removed the H9 at (49.8, 115.7)
- removed the H9 at (49.8, 80.2)
- removed the H9 at (92.2, 115.7)
- removed J10 (x4): T2, TestPoint:TestPoint_Pad_1.0x1.0mm
- removed J12 (x4): 12V, TestPoint:TestPoint_Pad_1.0x1.0mm
- removed J2 (x3): PRI, TerminalBlock:TerminalBlock_bornier-2_P5.08mm
- removed the J4 at (204.6, 145.5)
- removed the J4 at (204.6, 90.7)
- removed the J4 at (204.6, 118.1)
- removed the J6 at (204.6, 92.8)
- removed the J6 at (204.6, 147.6)
- removed the J6 at (204.6, 120.2)
- removed the J8 at (184.2, 128.5)
- removed the J8 at (184.2, 73.7)
- removed the J8 at (184.2, 101.1)
- removed J9 (x3): T1, TestPoint:TestPoint_Pad_1.0x1.0mm
- removed the L1 at (100.9, 117.0)
- removed the L1 at (100.9, 81.5)
- removed the L1 at (58.5, 117.0)
- removed the L1 at (58.5, 81.5)
- removed the L2 at (159.3, 92.3)
- removed the L2 at (159.3, 147.1)
- removed the L2 at (159.3, 119.7)
- removed the L3 at (159.3, 106.7)
- removed the L3 at (159.3, 134.1)
- removed the L3 at (159.3, 79.3)
- removed the Q1 at (170.1, 120.2)
- removed the Q1 at (170.1, 92.8)
- removed the Q1 at (170.1, 147.6)
- removed the Q2 at (170.2, 78.8)
- removed the Q2 at (170.2, 106.2)
- removed the Q2 at (170.2, 133.6)
- removed the Q3 at (190.7, 147.7)
- removed the Q3 at (190.7, 92.9)
- removed the Q3 at (190.7, 120.3)
- removed the R1 at (58.1, 102.5)
- removed the R1 at (100.5, 138.0)
- removed the R1 at (100.5, 102.5)
- removed the R1 at (58.1, 138.0)
- removed R10 (x4): 47k, Resistor_SMD:R_0805_2012Metric
- removed R11 (x4): 1k, Resistor_SMD:R_0805_2012Metric
- removed the R2 at (100.5, 98.9)
- removed the R2 at (100.5, 134.4)
- removed the R2 at (58.1, 134.4)
- removed the R2 at (58.1, 98.9)
- removed the R3 at (55.2, 98.9)
- removed the R3 at (97.6, 134.4)
- removed the R3 at (97.6, 98.9)
- removed the R3 at (55.2, 134.4)
- removed the R4 at (165.8, 111.8)
- removed the R4 at (93.9, 39.6)
- removed the R4 at (165.8, 139.2)
- removed the R4 at (165.8, 84.4)
- removed the R5 at (175.2, 84.4)
- removed the R5 at (175.2, 139.2)
- removed the R5 at (175.2, 111.8)
- removed the R5 at (103.2, 39.6)
- removed the R6 at (178.9, 111.8)
- removed the R6 at (106.9, 39.6)
- removed the R6 at (178.9, 139.2)
- removed the R6 at (178.9, 84.4)
- removed the R7 at (196.4, 114.8)
- removed the R7 at (196.4, 87.4)
- removed the R7 at (196.4, 142.2)
- removed the R8 at (196.5, 84.9)
- removed the R8 at (196.5, 112.3)
- removed the R8 at (196.5, 139.7)
- removed R9 (x4): 470, Resistor_SMD:R_0805_2012Metric
- removed the RV1 at (192.4, 77.5)
- removed the RV1 at (192.4, 132.3)
- removed the RV1 at (120.5, 32.8)
- removed the RV1 at (192.4, 104.9)
- removed the RV2 at (203.0, 132.3)
- removed the RV2 at (131.1, 32.8)
- removed the RV2 at (203.0, 104.9)
- removed the RV2 at (203.0, 77.5)
- removed the U1 at (61.5, 91.0)
- removed the U1 at (103.8, 91.0)
- removed the U1 at (103.8, 126.5)
- removed the U1 at (61.5, 126.5)
- removed the U2 at (202.5, 114.1)
- removed the U2 at (202.5, 141.5)
- removed the U2 at (202.5, 86.7)
- removed mouse-bite-2mm-slot (x10), mouse-bite-2mm-slot1 (x16), mouse-bite-2mm-slot2 (x16), mouse-bite-2mm-slot3 (x4), mouse-bite-2mm-slot4 (x4), mouse-bite-2mm-slot5 (x16): VAL**, Library:mouse-bite-2mm-slot
- added C15: 1u 100V, Capacitor_SMD:C_1206_3216Metric, F.Cu at (120.1, 37.6)
- added C8: 1000u, Capacitor_THT:CP_Radial_D16.0mm_P7.50mm, F.Cu at (34.5, 43.3)
- added D10: 180V, Diode_SMD:D_SMB, F.Cu at (118.9, 48.8)
- added D2: 180V, Diode_SMD:D_SMB, F.Cu at (93.0, 43.9)
- added D3: 180V, Diode_SMD:D_SMB, F.Cu at (93.0, 35.1)
- added D6: 1N5819, Diode_SMD:D_SOD-123, F.Cu at (113.3, 48.8)
- added D7: 1N5819, Diode_SMD:D_SOD-123, F.Cu at (109.2, 34.3)
- added D8: 1N4148, Diode_SMD:D_SOD-123, F.Cu at (132.6, 36.8)
- added D9: 1N4148, Diode_SMD:D_SOD-123, F.Cu at (135.1, 36.8)
- added G***: LOGO, LOGO, B.Cu at (120.7, 42.2)
- added J6: T2, TestPoint:TestPoint_Pad_1.0x1.0mm, F.Cu at (105.2, 34.3)
- added R4: 47k, Resistor_SMD:R_0805_2012Metric, F.Cu at (129.5, 32.6)
- added R5: 470, Resistor_SMD:R_0805_2012Metric, F.Cu at (134.6, 33.3)
- added R6: 1k, Resistor_SMD:R_0805_2012Metric, F.Cu at (131.3, 45.0)
- added RV1: 10k, Potentiometer_THT:Potentiometer_Bourns_3296W_Vertical, F.Cu at (114.9, 36.3)
- added RV2: 100k, Potentiometer_THT:Potentiometer_ACP_CA9-H2,5_Horizontal, F.Cu at (121.0, 30.0)
- added RV3: 10k, Potentiometer_THT:Potentiometer_ACP_CA9-H2,5_Horizontal, F.Cu at (131.9, 30.0)
- C9: renamed from C8; moved to B.Cu
- G***: moved to F.Cu
- H7: renamed from H4; value GND -> 12V
- J4: renamed from J8; moved to B.Cu
- moved G*** 37.5 mm to (77.7, 28.2)
- moved G*** 26.9 mm to (103.9, 39.6)
- moved J4 24.1 mm to (88.3, 26.7), turned to -90 degrees
- moved C9 16.7 mm to (92.1, 26.7), turned to 0 degrees
- moved G*** 16.7 mm to (126.0, 50.8)
- moved C12 8.49 mm to (129.5, 34.8), turned to 180 degrees
- moved C13 7.85 mm to (133.1, 40.5)
- moved C11 6.99 mm to (96.5, 35.1), turned to -90 degrees
- moved C16 6.57 mm to (138.2, 38.2), turned to 0 degrees
- moved D5 5.84 mm to (109.2, 29.0)
- moved Q2 5.75 mm to (100.9, 29.0)
- moved Q3 5.55 mm to (117.8, 42.7)
- moved R8 4.88 mm to (125.5, 45.0)
- moved U2 4.49 mm to (127.5, 38.6)
- moved J5 4.23 mm to (113.3, 52.6)
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- renumbered C2 to C1, C9 to C10, C10 to C11, C17 to C12, C14 to C13, C15 to C14, C3 to C2, C6 to C3, C1 to C4, C7 to C5, C4 to C6, C5 to C7, D3 to D4, D4 to D5, H11 to H1, H7 to H10, H8 to H11, H9 to H2, H10 to H3, H1 to H4, H2 to H5, H3 to H6, H5 to H8, H6 to H9, J2 to J1, J9 to J5, J4 to J7, J6 to J8, L2 to L1, L3 to L2, L1 to L3
Connections:
- net Net-(R7-Pad2) renamed interrupter
- C10 pad 2: Net-(C10-Pad2) -> GND
- C11 pad 2: Net-(C10-Pad2) -> GND
- C9 pad 2: Net-(C10-Pad2) -> GND
- D4 pad 1: Net-(C10-Pad2) -> GND
- D5 pad 1: Net-(C10-Pad2) -> GND
- H7 pad 1: GND -> +12V
- Q1 pad 3: Net-(C10-Pad2) -> GND
- Q2 pad 3: Net-(C10-Pad2) -> GND
- Q3 pad 2: Net-(C10-Pad2) -> Net-(C15-Pad1)
Routing:
- net Net-(C16-Pad1): track 106.0 -> 7.66 mm, vias 8 -> 0
- net Net-(D8-Pad2): track 114.2 -> 26.6 mm, vias 4 -> 0
- net Net-(R10-Pad1): track 70.1 -> 0.00 mm, vias 4 -> 0
- net Net-(Q3-Pad1): track 67.3 -> 0.00 mm, vias 8 -> 0
- net Net-(R9-Pad2): track 27.3 -> 0.00 mm
- net Net-(C14-Pad1): track 29.7 -> 10.7 mm
- net +12V: track 37.1 -> 55.3 mm, vias 4 -> 1
- net Net-(C13-Pad1): track 19.3 -> 2.16 mm
- net Net-(C15-Pad1): track 0.00 -> 11.3 mm
- net Net-(D6-Pad1): track 9.22 -> 0.00 mm
- net Net-(R5-Pad1): track 0.00 -> 7.38 mm
- net Net-(R4-Pad1): track 0.00 -> 7.29 mm
- net Net-(D5-Pad2): track 0.00 -> 6.83 mm
- net interrupter: track 11.0 -> 6.62 mm
- net Net-(D9-Pad1): track 0.00 -> 2.49 mm
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- added copper zone on F.Cu, net Net-(C15-Pad1)
- added copper zone on B.Cu, net Net-(C9-Pad1)
- added copper zone on F.Cu, net Net-(Q3-Pad1)
- removed copper zone on F.Cu, net (none)
- removed copper zone on B.Cu, net Net-(C10-Pad2)
- removed copper zone on F.Cu, net Net-(C10-Pad2)
- removed copper zone on F.Cu, net Net-(C9-Pad1)
- removed copper zone on B.Cu, net Net-(D2-Pad1)
- removed copper zone on F.Cu, net Net-(D2-Pad1)
Other:
- board size 203.6 x 138.7 mm -> 118.6 x 33.5 mm

Commit message: final clean-up
Parts:
- removed the G*** at (126.0, 50.8)
- removed the G*** at (103.9, 39.6)
- removed the G*** at (77.7, 28.2)
- removed the G*** at (52.3, 47.1)
- removed the G*** at (120.7, 42.2)
